File: kicad/kicad.kicad_pcb (KiCad board)
At the start: 2 copper layers, 55 x 105 mm, 12 parts, among them K1 RP1A23D5, U1 WeMos_D1_mini, X1 250-202, X2 250-202, X3 250-203

Commit message: Small schematic & footprint cleanups
Connections:
- net Net-(K1-Pad1) renamed /L
- net Net-(K1-Pad2) renamed /L_OUT
- net Net-(K1-Pad4) renamed GND
- net Net-(PS1-Pad1) renamed /N
Routing:
- net /N: track 83.1 -> 71.5 mm
- net /L: track 34.2 -> 40.0 mm
Other:
- board text added: "Proofer box temperature controller - V1.1"
- board text removed: "Proofer box temperature controller - V1.0"

Commit message: WIP: some more schematic & footprint updates
Parts:
- R1: footprint Resistor_THT:R_Axial_DIN0207_L6.3mm_D2.5mm_P7.62mm_Horizontal -> Resistor_THT:R_Axial_DIN0207_L6.3mm_D2.5mm_P10.16mm_Horizontal
- moved R1 2.54 mm to (204.7, 30.5)
Connections:
- net /L renamed L
- net /L_OUT renamed L_OUT
- net /N renamed N
- net Net-(R1-Pad1) renamed 3V3
- net Net-(R1-Pad2) renamed DATA
Routing:
- net 3V3: track 39.8 -> 41.3 mm
